Commit message: Rviz Complete

File: leg_description/urdf/my_leg.xacro (robot description, xacro)
@@ -1,15 +1,29 @@
 <?xml version="1.0"?>
 <robot xmlns:xacro="http://www.ros.org/wiki/xacro" name="RR">
+<material name="blue">
+  <color rgba="0 0 0.8 1"/>
+</material>
+<material name="red">
+  <color rgba="0.8 0 0 1"/>
+</material>
+<material name="grey">
+  <color rgba="0.5 0.5 0.5 1"/>
+</material>
+<material name="DarkGrey">
+  <color rgba="0.3 0.3 0.3 1"/>
+</material>
 <!-- Defining macros -->
-<xacro:property name="box_X" value="0.2" />
-<xacro:property name="box_Y" value="0.2" />
-<xacro:property name="box_Z" value="0.5" />
+<xacro:property name="BaseHeight" value="0.5" />
 <!-- Actuator -->
+<xacro:property name="actuator_nudge" value="0.00666" />
+<xacro:property name="actuator_cylinder_width" value="0.03084" />
 <xacro:property name="actuator_total_width" value="0.05708" />
 <xacro:property name="actuator_diameter" value="0.1031" />
-<xacro:property name="bodylen" value="1" />
-<xacro:property name="height" value="0.1" />
-<xacro:property name="offset" value="0.1" />
-<xacro:property name="base_height" value="1" />
+<!-- "actuator_offset_from_peripheral_connector" -> AOFPC -->
+<xacro:property name="AOFPC" value="0.05755" />
+<!-- Link2 -->
+<xacro:property name="link1_2D" value="0.089" />
+<!-- Link3 -->
+<xacro:property name="link2_3D" value="0.337" />
 <!-- Moment of inertia -->
 <xacro:macro name="default_inertial" params="mass xl yl zl *Dorigin">
@@ -22,49 +36,14 @@
     </inertial>
 </xacro:macro>
-<material name="blue">
-  <color rgba="0 0 0.8 1"/>
-</material>
-<material name="red">
-  <color rgba="0.8 0 0 1"/>
-</material>
 <!-- Addin objects: -->
 <link name="world"/>
- <joint name="world_joint" type="fixed">
-  <parent link="world"/>
-  <child link="base_link"/>
-  <origin rpy="0 ${-pi/2} ${-pi/2}" xyz="0 0 ${box_Z}"/>
-</joint>
-<!-- <link name="base_link">
-  <visual>
-    <geometry>
-      <box size="${box_X} ${box_Y} ${box_Z}"/>
-    </geometry>
-    <origin rpy="0 0 0" xyz="0 0 ${-box_Z/2}"/>
-    <material name="blue"/>
-  </visual>
-  <collision>
-    <geometry>
-      <box size="${box_X} ${box_Y} ${box_Z}"/>
-    </geometry>
-    <origin rpy="0 0 0" xyz="0 0 ${-box_Z/2}"/>
-  </collision>
-  <inertial>
-    <mass value="100" />
-    <inertia ixx="0.0100" ixy="0.0" ixz="0.0"
-              iyy="0.0100" iyz="0.0"
-              izz="0.0100" />
-    <origin rpy="0 0 0" xyz="0 0 ${-base_height/2}"/>
-  </inertial>
-</link>
- -->
-<!-- Link 1  -->
+<!-- Base Link  -->
 <link name="base_link">
   <visual>
     <geometry>
-        <mesh scale=".001 .001 .001" filename="package://leg_description/meshes/link2stl.STL" />
+        <mesh scale=".001 .001 .001" filename="package://leg_description/meshes/Base.STL" />
     </geometry>
-    <origin rpy="0 0 0" xyz="${-actuator_diameter/2} ${-actuator_diameter/2} 0"/>
-    <!-- <origin rpy="0 ${-pi/2} ${-pi/2}" xyz="0 0 0"/> -->
-    <material name="red"/>
+    <origin rpy="0 0 0" xyz="0 0 0"/>
+    <material name="DarkGrey"/>
   </visual>
   <collision>
@@ -78,13 +57,18 @@
   </xacro:default_inertial>
 </link>
+ <joint name="world_joint" type="fixed">
+  <parent link="world"/>
+  <child link="base_link"/>
+  <origin rpy="0 ${-pi/2} ${-pi/2}" xyz="${AOFPC} 0 ${BaseHeight}"/>
+</joint>
 <!-- Link 1  -->
-<!-- <link name="link1">
+<link name="link1">
   <visual>
     <geometry>
-        <mesh scale=".001 .001 .001" filename="package://leg_description/meshes/link2stl.STL" />
+        <mesh scale=".001 .001 .001" filename="package://leg_description/meshes/link1.STL" />
     </geometry>
     <origin rpy="0 0 0" xyz="0 0 0"/>
-    <origin rpy="0 ${-pi/2} ${-pi/2}" xyz="0 0 0"/>
-    <material name="red"/>
+    <!-- <origin rpy="0 ${-pi/2} ${-pi/2}" xyz="0 0 0"/> -->
+    <material name="grey"/>
   </visual>
   <collision>
@@ -102,5 +86,55 @@
   <child link="link1"/>
   <axis rpy = "0 0 0" xyz="0 0 1"/>
-  <origin rpy = "0 0 0" xyz="0 0 ${actuator_total_width/2}"/>
-</joint>   -->
+  <origin rpy = "${pi} 0 0" xyz="0 0 ${actuator_cylinder_width/2+actuator_nudge +AOFPC}"/>
+</joint>
+<!-- Link 2  -->
+<link name="link2">
+  <visual>
+    <geometry>
+        <mesh scale=".001 .001 .001" filename="package://leg_description/meshes/link2stl.STL" />
+    </geometry>
+    <origin rpy="0 0 0" xyz="0 0 0"/>
+    <material name="DarkGrey"/>
+  </visual>
+  <collision>
+    <geometry>
+      <cylinder radius="${actuator_diameter}" length="${actuator_total_width}"/>
+    </geometry>
+    <origin rpy="${pi/2} 0 ${-pi/2}" xyz="0 0 0"/>
+  </collision>
+  <xacro:default_inertial mass="10" xl="1" yl="1" zl="1">
+    <origin rpy="0 0 0" xyz="0 0 0" />
+  </xacro:default_inertial>
+</link>
+<joint name="link1_to_link2" type="continuous">
+  <parent link="link1"/>
+  <child link="link2"/>
+  <axis rpy = "0 0 0" xyz="0 0 1"/>
+  <origin rpy = "${pi/2} ${pi/2} 0" xyz="0 ${-(  actuator_cylinder_width/2+actuator_nudge +link1_2D)}  0"/>
+</joint>
+<!-- Link 3  -->
+<link name="link3">
+  <visual>
+    <geometry>
+        <mesh scale=".001 .001 .001" filename="package://leg_description/meshes/link3stl.STL" />
+    </geometry>
+    <origin rpy="0 0 0" xyz="0 0 0"/>
+    <material name="grey"/>
+  </visual>
+  <collision>
+    <geometry>
+      <cylinder radius="${actuator_diameter}" length="${actuator_total_width}"/>
+    </geometry>
+    <origin rpy="${pi/2} 0 ${-pi/2}" xyz="0 0 0"/>
+  </collision>
+  <xacro:default_inertial mass="10" xl="1" yl="1" zl="1">
+    <origin rpy="0 0 0" xyz="0 0 0" />
+  </xacro:default_inertial>
+</link>
+<joint name="link2_to_link3" type="continuous">
+  <parent link="link2"/>
+  <child link="link3"/>
+  <axis rpy = "0 0 0" xyz="0 0 1"/>
+  <origin rpy = "0 0 0" xyz="${link2_3D} 0  0"/>
+</joint>
 </robot>

Commit message: Imported the model to gazebo

File: leg_description/urdf/my_leg.xacro (robot description, xacro)
@@ -1,4 +1,5 @@
 <?xml version="1.0"?>
 <robot xmlns:xacro="http://www.ros.org/wiki/xacro" name="RR">
+<!-- Colors -->
 <material name="blue">
   <color rgba="0 0 0.8 1"/>
@@ -22,8 +23,12 @@
 <!-- "actuator_offset_from_peripheral_connector" -> AOFPC -->
 <xacro:property name="AOFPC" value="0.05755" />
+<!-- Actuator Limits -->
+<xacro:property name="velocity_limit" value="398" />
+<xacro:property name="effort_limit" value="0.8844" />
 <!-- Link2 -->
 <xacro:property name="link1_2D" value="0.089" />
 <!-- Link3 -->
 <xacro:property name="link2_3D" value="0.337" />
+<xacro:property name="link3_angle_limit" value="2.15" />
 <!-- Moment of inertia -->
 <xacro:macro name="default_inertial" params="mass xl yl zl *Dorigin">
@@ -82,10 +87,20 @@
   </xacro:default_inertial>
 </link>
-<joint name="base_to_link1" type="continuous">
+<joint name="base_to_link1" type="revolute">
   <parent link="base_link"/>
   <child link="link1"/>
   <axis rpy = "0 0 0" xyz="0 0 1"/>
+  <limit lower="${-pi/2}" upper="${pi/2}" effort="${effort_limit}" velocity="${velocity_limit}" />
   <origin rpy = "${pi} 0 0" xyz="0 0 ${actuator_cylinder_width/2+actuator_nudge +AOFPC}"/>
 </joint>
+<transmission name="base_link1_trans">
+    <type>transmission_interface/SimpleTransmission</type>
+    <actuator name="$motor1">
+      <mechanicalReduction>7</mechanicalReduction>
+    </actuator>
+    <joint name="base_to_link1">
+      <hardwareInterface>hardware_interface/EffortJointInterface</hardwareInterface>
+    </joint>
+  </transmission>
 <!-- Link 2  -->
 <link name="link2">
@@ -113,4 +128,13 @@
   <origin rpy = "${pi/2} ${pi/2} 0" xyz="0 ${-(  actuator_cylinder_width/2+actuator_nudge +link1_2D)}  0"/>
 </joint>
+<transmission name="link1_link2_trans">
+    <type>transmission_interface/SimpleTransmission</type>
+    <actuator name="$motor2">
+      <mechanicalReduction>10</mechanicalReduction>
+    </actuator>
+    <joint name="link1_to_link2">
+      <hardwareInterface>hardware_interface/EffortJointInterface</hardwareInterface>
+    </joint>
+  </transmission>
 <!-- Link 3  -->
 <link name="link3">
@@ -132,9 +156,25 @@
   </xacro:default_inertial>
 </link>
-<joint name="link2_to_link3" type="continuous">
+<joint name="link2_to_link3" type="revolute">
   <parent link="link2"/>
   <child link="link3"/>
   <axis rpy = "0 0 0" xyz="0 0 1"/>
   <origin rpy = "0 0 0" xyz="${link2_3D} 0  0"/>
+  <limit lower="${-link3_angle_limit}" upper="${link3_angle_limit}" effort="${effort_limit}" velocity="${velocity_limit}" />
 </joint>
+<transmission name="link2_link3_trans">
+    <type>transmission_interface/SimpleTransmission</type>
+    <actuator name="$motor3">
+      <mechanicalReduction>10</mechanicalReduction>
+    </actuator>
+    <joint name="link2_to_link3">
+      <hardwareInterface>hardware_interface/EffortJointInterface</hardwareInterface>
+    </joint>
+  </transmission>
+<!-- Gazebo -->
+<gazebo>
+    <plugin name="gazebo_ros_control" filename="libgazebo_ros_control.so">
+      <robotNamespace>/leg</robotNamespace>
+    </plugin>
+</gazebo>
 </robot>

Commit message: inserted Leg collision elements

File: leg_description/urdf/my_leg.xacro (robot description, xacro)
@@ -16,4 +16,6 @@
 <!-- Defining macros -->
 <xacro:property name="BaseHeight" value="0.5" />
+<!-- Connectors -->
+<xacro:property name="Connector1_L" value="0.006" />
 <!-- Actuator -->
 <xacro:property name="actuator_nudge" value="0.00666" />
@@ -21,9 +23,11 @@
 <xacro:property name="actuator_total_width" value="0.05708" />
 <xacro:property name="actuator_diameter" value="0.1031" />
-<!-- "actuator_offset_from_peripheral_connector" -> AOFPC -->
-<xacro:property name="AOFPC" value="0.05755" />
 <!-- Actuator Limits -->
 <xacro:property name="velocity_limit" value="398" />
 <xacro:property name="effort_limit" value="0.8844" />
+<!-- Generated Quantities -->
+<xacro:property name="actuator_midplane_origin_offset" value="${(actuator_total_width-actuator_cylinder_width)/2}" />
+<!-- "actuator_offset_from_peripheral_connector" -> AOFPC -->
+<xacro:property name="AOFPC" value="${actuator_diameter/2+Connector1_L}" />
 <!-- Link2 -->
 <xacro:property name="link1_2D" value="0.089" />
@@ -31,4 +35,6 @@
 <xacro:property name="link2_3D" value="0.337" />
 <xacro:property name="link3_angle_limit" value="2.15" />
+<xacro:property name="link3_ED" value="0.369" />
+<xacro:property name="footD" value="0.050" />
 <!-- Moment of inertia -->
 <xacro:macro name="default_inertial" params="mass xl yl zl *Dorigin">
@@ -54,7 +60,7 @@
   <collision>
     <geometry>
-      <cylinder radius="${actuator_diameter}" length="${actuator_total_width}"/>
+      <cylinder radius="${actuator_diameter/2+Connector1_L}" length="${actuator_total_width}"/>
     </geometry>
-    <origin rpy="${pi/2} 0 ${-pi/2}" xyz="0 0 0"/>
+    <origin rpy="0 0 0" xyz="0 ${actuator_midplane_origin_offset/2} 0"/>
   </collision>
   <xacro:default_inertial mass="10" xl="1" yl="1" zl="1">
@@ -74,12 +80,11 @@
     </geometry>
     <origin rpy="0 0 0" xyz="0 0 0"/>
-    <!-- <origin rpy="0 ${-pi/2} ${-pi/2}" xyz="0 0 0"/> -->
     <material name="grey"/>
   </visual>
   <collision>
     <geometry>
-      <cylinder radius="${actuator_diameter}" length="${actuator_total_width}"/>
+      <cylinder radius="${actuator_diameter/2+Connector1_L}" length="${actuator_total_width}"/>
     </geometry>
-    <origin rpy="${pi/2} 0 ${-pi/2}" xyz="0 0 0"/>
+    <origin rpy="${pi/2} 0 0" xyz="0  ${actuator_midplane_origin_offset/2} 0"/>
   </collision>
   <xacro:default_inertial mass="10" xl="1" yl="1" zl="1">
@@ -114,7 +119,7 @@
   <collision>
     <geometry>
-      <cylinder radius="${actuator_diameter}" length="${actuator_total_width}"/>
+      <cylinder radius="0.025" length="${link2_3D}"/>
     </geometry>
-    <origin rpy="${pi/2} 0 ${-pi/2}" xyz="0 0 0"/>
+    <origin rpy="0 ${pi/2} 0" xyz="${link2_3D /2} 0 0"/>
   </collision>
   <xacro:default_inertial mass="10" xl="1" yl="1" zl="1">
@@ -146,9 +151,15 @@
     <material name="grey"/>
   </visual>
-  <collision>
+  <collision name="link3_leg">
     <geometry>
-      <cylinder radius="${actuator_diameter}" length="${actuator_total_width}"/>
+      <cylinder radius="0.025" length="${link3_ED- (footD/2) }"/>
     </geometry>
-    <origin rpy="${pi/2} 0 ${-pi/2}" xyz="0 0 0"/>
+    <origin rpy="0 ${pi/2} 0" xyz="${( link3_ED- footD/2 )/2  } 0 0"/>
+  </collision>
+  <collision name="link3_foot">
+    <geometry>
+      <sphere radius="${footD/2}"/>
+    </geometry>
+    <origin rpy="0 0 0" xyz="${ link3_ED- footD/2  } 0 0"/>
   </collision>
   <xacro:default_inertial mass="10" xl="1" yl="1" zl="1">

Commit message: fixed base collision

File: leg_description/urdf/my_leg.xacro (robot description, xacro)
@@ -62,5 +62,5 @@
       <cylinder radius="${actuator_diameter/2+Connector1_L}" length="${actuator_total_width}"/>
     </geometry>
-    <origin rpy="0 0 0" xyz="0 ${actuator_midplane_origin_offset/2} 0"/>
+    <origin rpy="0 0 0" xyz="0 0 ${-actuator_midplane_origin_offset/2}"/>
   </collision>
   <xacro:default_inertial mass="10" xl="1" yl="1" zl="1">
@@ -164,5 +164,5 @@
   </collision>
   <xacro:default_inertial mass="10" xl="1" yl="1" zl="1">
-    <origin rpy="0 0 0" xyz="0 0 0" />
+    <origin rpy="0 0 0" xyz="${link3_ED/2} 0 0" />
   </xacro:default_inertial>
 </link>

Commit message: added knee and link2unit collision geometries

File: leg_description/urdf/my_leg.xacro (robot description, xacro)
@@ -17,5 +17,12 @@
 <xacro:property name="BaseHeight" value="0.5" />
 <!-- Connectors -->
-<xacro:property name="Connector1_L" value="0.006" />
+<xacro:property name="connectorL_1" value="0.006" />
+<xacro:property name="connectorL_2" value="0.027" />
+<!-- Hip -->
+<xacro:property name="hipW" value="0.049" />
+<!-- Knee -->
+<xacro:property name="knee_gearD" value="0.05" />
+<!-- foot -->
+<xacro:property name="legD" value="0.05" />
 <!-- Actuator -->
 <xacro:property name="actuator_nudge" value="0.00666" />
@@ -29,5 +36,6 @@
 <xacro:property name="actuator_midplane_origin_offset" value="${(actuator_total_width-actuator_cylinder_width)/2}" />
 <!-- "actuator_offset_from_peripheral_connector" -> AOFPC -->
-<xacro:property name="AOFPC" value="${actuator_diameter/2+Connector1_L}" />
+<xacro:property name="AOFPC" value="${actuator_diameter/2+connectorL_1}" />
+<xacro:property name="actuator3_wt_connectorL" value="${actuator_cylinder_width+connectorL_2+actuator_nudge}" />
 <!-- Link2 -->
 <xacro:property name="link1_2D" value="0.089" />
@@ -60,5 +68,5 @@
   <collision>
     <geometry>
-      <cylinder radius="${actuator_diameter/2+Connector1_L}" length="${actuator_total_width}"/>
+      <cylinder radius="${actuator_diameter/2+connectorL_1}" length="${actuator_total_width}"/>
     </geometry>
     <origin rpy="0 0 0" xyz="0 0 ${-actuator_midplane_origin_offset/2}"/>
@@ -84,5 +92,5 @@
   <collision>
     <geometry>
-      <cylinder radius="${actuator_diameter/2+Connector1_L}" length="${actuator_total_width}"/>
+      <cylinder radius="${actuator_diameter/2+connectorL_1}" length="${actuator_total_width}"/>
     </geometry>
     <origin rpy="${pi/2} 0 0" xyz="0  ${actuator_midplane_origin_offset/2} 0"/>
@@ -117,9 +125,15 @@
     <material name="DarkGrey"/>
   </visual>
-  <collision>
-    <geometry>
-      <cylinder radius="0.025" length="${link2_3D}"/>
+  <collision name="link2_leg">
+    <geometry>
+      <cylinder radius="${legD/2}" length="${link2_3D}"/>
     </geometry>
     <origin rpy="0 ${pi/2} 0" xyz="${link2_3D /2} 0 0"/>
+  </collision>
+  <collision name="link2_unit">
+    <geometry>
+      <cylinder radius="${actuator_diameter/2+connectorL_1}" length="${hipW+actuator3_wt_connectorL}"/>
+    </geometry>
+    <origin rpy="0 0 0" xyz="0 0 ${-(actuator3_wt_connectorL/2)}"/>
   </collision>
   <xacro:default_inertial mass="10" xl="1" yl="1" zl="1">
@@ -153,7 +167,13 @@
   <collision name="link3_leg">
     <geometry>
-      <cylinder radius="0.025" length="${link3_ED- (footD/2) }"/>
+      <cylinder radius="${legD/2}" length="${link3_ED- (footD/2) }"/>
     </geometry>
     <origin rpy="0 ${pi/2} 0" xyz="${( link3_ED- footD/2 )/2  } 0 0"/>
+  </collision>
+  <collision name="link3_knee">
+    <geometry>
+      <cylinder radius="${knee_gearD/2}" length="${legD }"/>
+    </geometry>
+    <origin rpy="0 0 0" xyz="0 0 0"/>
   </collision>
   <collision name="link3_foot">

Commit message: added updated stls

File: leg_description/urdf/my_leg.xacro (robot description, xacro)
@@ -17,12 +17,12 @@
 <xacro:property name="BaseHeight" value="0.5" />
 <!-- Connectors -->
-<xacro:property name="connectorL_1" value="0.006" />
-<xacro:property name="connectorL_2" value="0.027" />
+<xacro:property name="connectorL_1" value="0.004" />
+<xacro:property name="connectorL_2" value="0.030" />
 <!-- Hip -->
-<xacro:property name="hipW" value="0.049" />
+<xacro:property name="hipW" value="0.045" />
 <!-- Knee -->
 <xacro:property name="knee_gearD" value="0.05" />
 <!-- foot -->
-<xacro:property name="legD" value="0.05" />
+<xacro:property name="legD" value="0.045" />
 <!-- Actuator -->
 <xacro:property name="actuator_nudge" value="0.00666" />
@@ -32,5 +32,7 @@
 <!-- Actuator Limits -->
 <xacro:property name="velocity_limit" value="398" />
-<xacro:property name="effort_limit" value="0.8844" />
+<xacro:property name="maxCurrent" value="13.36" />
+<xacro:property name="motorConstantKt" value="0.8" />
+<xacro:property name="effort_limit" value="${maxCurrent*motorConstantKt}" />
 <!-- Generated Quantities -->
 <xacro:property name="actuator_midplane_origin_offset" value="${(actuator_total_width-actuator_cylinder_width)/2}" />
@@ -79,5 +81,5 @@
   <parent link="world"/>
   <child link="base_link"/>
-  <origin rpy="0 ${-pi/2} ${-pi/2}" xyz="${AOFPC} 0 ${BaseHeight}"/>
+  <origin rpy="${pi/2} ${-pi/2} 0" xyz="${AOFPC} 0 ${BaseHeight}"/>
 </joint>
 <!-- Link 1  -->
@@ -105,5 +107,5 @@
   <axis rpy = "0 0 0" xyz="0 0 1"/>
   <limit lower="${-pi/2}" upper="${pi/2}" effort="${effort_limit}" velocity="${velocity_limit}" />
-  <origin rpy = "${pi} 0 0" xyz="0 0 ${actuator_cylinder_width/2+actuator_nudge +AOFPC}"/>
+  <origin rpy = "0 0 0" xyz="0 0 ${-(actuator_cylinder_width/2+actuator_nudge +AOFPC)}"/>
 </joint>
 <transmission name="base_link1_trans">
@@ -120,5 +122,5 @@
   <visual>
     <geometry>
-        <mesh scale=".001 .001 .001" filename="package://leg_description/meshes/link2stl.STL" />
+        <mesh scale=".001 .001 .001" filename="package://leg_description/meshes/link2.STL" />
     </geometry>
     <origin rpy="0 0 0" xyz="0 0 0"/>
@@ -156,9 +158,9 @@
     </joint>
   </transmission>
-<!-- Link 3  -->
+  <!-- Link 3  -->
 <link name="link3">
   <visual>
     <geometry>
-        <mesh scale=".001 .001 .001" filename="package://leg_description/meshes/link3stl.STL" />
+        <mesh scale=".001 .001 .001" filename="package://leg_description/meshes/link3.STL" />
     </geometry>
     <origin rpy="0 0 0" xyz="0 0 0"/>
