Commit message: better_commbination_v1

File: leg_description/urdf/my_leg.xacro (robot description, xacro)
@@ -16,13 +16,16 @@
 <!-- Defining macros -->
 <xacro:property name="BaseHeight" value="0.5" />
+<!-- Lengths -->
+<xacro:property name="LB0" value="0.05555" />
+<xacro:property name="L01" value="0.07763" />
+<xacro:property name="L12" value="0.11208" />
+<xacro:property name="L23" value="0.2531" />
+<xacro:property name="L3E" value="0.248" />
 <!-- Connectors -->
 <xacro:property name="connectorL_1" value="0.004" />
-<xacro:property name="connectorL_2" value="0.030" />
 <!-- Hip -->
 <xacro:property name="hipW" value="0.045" />
-<!-- Knee -->
-<xacro:property name="knee_gearD" value="0.05" />
-<!-- foot -->
-<xacro:property name="legD" value="0.045" />
+<!-- leg -->
+<xacro:property name="legD" value="0.041" />
 <!-- Actuator -->
 <xacro:property name="actuator_nudge" value="0.00666" />
@@ -30,4 +33,9 @@
 <xacro:property name="actuator_total_width" value="0.05708" />
 <xacro:property name="actuator_diameter" value="0.1031" />
+<!-- Generated Quantities -->
+<!-- AMOO = "actuator_midplane_origin_offset" -->
+<xacro:property name="AMOO" value="${(actuator_total_width-actuator_cylinder_width)/2}" />
+<xacro:property name="link1_total_length" value="${-hipW/2 + L12 + actuator_total_width-(actuator_cylinder_width/2+actuator_nudge)}" />
+<xacro:property name="link1_total_mid_originL" value="${link1_total_length/2 - ( actuator_total_width - actuator_cylinder_width/2 - actuator_nudge) }" />
 <!-- Actuator Limits -->
 <xacro:property name="velocity_limit" value="398" />
@@ -35,16 +43,4 @@
 <xacro:property name="motorConstantKt" value="0.8" />
 <xacro:property name="effort_limit" value="${maxCurrent*motorConstantKt}" />
-<!-- Generated Quantities -->
-<xacro:property name="actuator_midplane_origin_offset" value="${(actuator_total_width-actuator_cylinder_width)/2}" />
-<!-- "actuator_offset_from_peripheral_connector" -> AOFPC -->
-<xacro:property name="AOFPC" value="${actuator_diameter/2+connectorL_1}" />
-<xacro:property name="actuator3_wt_connectorL" value="${actuator_cylinder_width+connectorL_2+actuator_nudge}" />
-<!-- Link2 -->
-<xacro:property name="link1_2D" value="0.089" />
-<!-- Link3 -->
-<xacro:property name="link2_3D" value="0.337" />
-<xacro:property name="link3_angle_limit" value="2.15" />
-<xacro:property name="link3_ED" value="0.369" />
-<xacro:property name="footD" value="0.050" />
 <!-- Moment of inertia -->
 <xacro:macro name="default_inertial" params="mass xl yl zl *Dorigin">
@@ -72,14 +68,22 @@
       <cylinder radius="${actuator_diameter/2+connectorL_1}" length="${actuator_total_width}"/>
     </geometry>
-    <origin rpy="0 0 0" xyz="0 0 ${-actuator_midplane_origin_offset/2}"/>
+    <origin rpy="0 0 0" xyz="0 0 ${AMOO/2}"/>
   </collision>
-  <xacro:default_inertial mass="10" xl="1" yl="1" zl="1">
-    <origin rpy="0 0 0" xyz="0 0 0" />
-  </xacro:default_inertial>
+  <inertial>
+    <mass value="1.14058" />
+    <inertia
+    ixx="0.000576572"
+    ixy="-1.091449e-05"
+    ixz="4.096e-06"
+    iyy="0.000825053"
+    iyz="3.018e-06"
+    izz="0.000391889" />
+    <origin rpy="0 0 0" xyz="-0.00083 -0.00061 0.01032" />
+  </inertial>
 </link>
- <joint name="world_joint" type="fixed">
+<joint name="world_joint" type="fixed">
   <parent link="world"/>
   <child link="base_link"/>
-  <origin rpy="${pi/2} ${-pi/2} 0" xyz="${AOFPC} 0 ${BaseHeight}"/>
+  <origin rpy="${pi/2} ${-pi/2} 0" xyz="${LB0} 0 ${BaseHeight}"/>
 </joint>
 <!-- Link 1  -->
@@ -94,11 +98,19 @@
   <collision>
     <geometry>
-      <cylinder radius="${actuator_diameter/2+connectorL_1}" length="${actuator_total_width}"/>
+      <cylinder radius="${actuator_diameter/2+connectorL_1}" length="${link1_total_length}"/>
     </geometry>
-    <origin rpy="${pi/2} 0 0" xyz="0  ${actuator_midplane_origin_offset/2} 0"/>
+    <origin rpy="${pi/2} 0 0" xyz="0  ${-link1_total_mid_originL} 0"/>
   </collision>
-  <xacro:default_inertial mass="10" xl="1" yl="1" zl="1">
-    <origin rpy="0 0 0" xyz="0 0 0" />
-  </xacro:default_inertial>
+  <inertial>
+    <mass value="1.14058" />
+    <inertia
+    ixx="0.000576572"
+    ixy="-1.091449e-05"
+    ixz="4.096e-06"
+    iyy="0.000825053"
+    iyz="3.018e-06"
+    izz="0.000391889" />
+    <origin rpy="0 0 0" xyz="-0.00083 -0.00061 0.01032" />
+  </inertial>
 </link>
 <joint name="base_to_link1" type="revolute">
@@ -107,5 +119,5 @@
   <axis rpy = "0 0 0" xyz="0 0 1"/>
   <limit lower="${-pi/2}" upper="${pi/2}" effort="${effort_limit}" velocity="${velocity_limit}" />
-  <origin rpy = "0 0 0" xyz="0 0 ${-(actuator_cylinder_width/2+actuator_nudge +AOFPC)}"/>
+  <origin rpy = "0 0 0" xyz="0 0 ${-L01}"/>
 </joint>
 <transmission name="base_link1_trans">
@@ -117,5 +129,5 @@
       <hardwareInterface>hardware_interface/EffortJointInterface</hardwareInterface>
     </joint>
-  </transmission>
+</transmission>
 <!-- Link 2  -->
 <link name="link2">
@@ -129,17 +141,25 @@
   <collision name="link2_leg">
     <geometry>
-      <cylinder radius="${legD/2}" length="${link2_3D}"/>
+      <cylinder radius="${legD/2}" length="${L23}"/>
     </geometry>
-    <origin rpy="0 ${pi/2} 0" xyz="${link2_3D /2} 0 0"/>
+    <origin rpy="0 ${pi/2} 0" xyz="${L23/2} 0 0"/>
   </collision>
-  <collision name="link2_unit">
+  <!-- <collision name="link2_unit">
     <geometry>
       <cylinder radius="${actuator_diameter/2+connectorL_1}" length="${hipW+actuator3_wt_connectorL}"/>
     </geometry>
     <origin rpy="0 0 0" xyz="0 0 ${-(actuator3_wt_connectorL/2)}"/>
-  </collision>
-  <xacro:default_inertial mass="10" xl="1" yl="1" zl="1">
-    <origin rpy="0 0 0" xyz="0 0 0" />
-  </xacro:default_inertial>
+  </collision> -->
+  <inertial>
+    <mass value="0.94987" />
+    <inertia
+    ixx="0.001561735"
+    ixy="1.2537e-05"
+    ixz="0.000843757"
+    iyy="0.005174717"
+    iyz="1.72e-05"
+    izz="0.004776989" />
+    <origin rpy="0 0 0" xyz="0.03158 -0.00042 -0.02813" />
+  </inertial>
 </link>
 <joint name="link1_to_link2" type="continuous">
@@ -147,5 +167,5 @@
   <child link="link2"/>
   <axis rpy = "0 0 0" xyz="0 0 1"/>
-  <origin rpy = "${pi/2} ${pi/2} 0" xyz="0 ${-(  actuator_cylinder_width/2+actuator_nudge +link1_2D)}  0"/>
+  <origin rpy = "${pi/2} ${pi/2} 0" xyz="0 ${-L12}  0"/>
 </joint>
 <transmission name="link1_link2_trans">
@@ -158,51 +178,4 @@
     </joint>
   </transmission>
-  <!-- Link 3  -->
-<link name="link3">
-  <visual>
-    <geometry>
-        <mesh scale=".001 .001 .001" filename="package://leg_description/meshes/link3.STL" />
-    </geometry>
-    <origin rpy="0 0 0" xyz="0 0 0"/>
-    <material name="grey"/>
-  </visual>
-  <collision name="link3_leg">
-    <geometry>
-      <cylinder radius="${legD/2}" length="${link3_ED- (footD/2) }"/>
-    </geometry>
-    <origin rpy="0 ${pi/2} 0" xyz="${( link3_ED- footD/2 )/2  } 0 0"/>
-  </collision>
-  <collision name="link3_knee">
-    <geometry>
-      <cylinder radius="${knee_gearD/2}" length="${legD }"/>
-    </geometry>
-    <origin rpy="0 0 0" xyz="0 0 0"/>
-  </collision>
-  <collision name="link3_foot">
-    <geometry>
-      <sphere radius="${footD/2}"/>
-    </geometry>
-    <origin rpy="0 0 0" xyz="${ link3_ED- footD/2  } 0 0"/>
-  </collision>
-  <xacro:default_inertial mass="10" xl="1" yl="1" zl="1">
-    <origin rpy="0 0 0" xyz="${link3_ED/2} 0 0" />
-  </xacro:default_inertial>
-</link>
-<joint name="link2_to_link3" type="revolute">
-  <parent link="link2"/>
-  <child link="link3"/>
-  <axis rpy = "0 0 0" xyz="0 0 1"/>
-  <origin rpy = "0 0 0" xyz="${link2_3D} 0  0"/>
-  <limit lower="${-link3_angle_limit}" upper="${link3_angle_limit}" effort="${effort_limit}" velocity="${velocity_limit}" />
-</joint>
-<transmission name="link2_link3_trans">
-    <type>transmission_interface/SimpleTransmission</type>
-    <actuator name="$motor3">
-      <mechanicalReduction>10</mechanicalReduction>
-    </actuator>
-    <joint name="link2_to_link3">
-      <hardwareInterface>hardware_interface/EffortJointInterface</hardwareInterface>
-    </joint>
-  </transmission>
 <!-- Gazebo -->
 <gazebo>

Commit message: final model (without inertia of rotor and belt)

File: leg_description/urdf/my_leg.xacro (robot description, xacro)
@@ -15,5 +15,5 @@
 </material>
 <!-- Defining macros -->
-<xacro:property name="BaseHeight" value="0.5" />
+<xacro:property name="BaseHeight" value="0.4" />
 <!-- Lengths -->
 <xacro:property name="LB0" value="0.05555" />
@@ -21,11 +21,19 @@
 <xacro:property name="L12" value="0.11208" />
 <xacro:property name="L23" value="0.2531" />
-<xacro:property name="L3E" value="0.248" />
+<xacro:property name="L3E" value="0.2455" />
 <!-- Connectors -->
 <xacro:property name="connectorL_1" value="0.004" />
 <!-- Hip -->
 <xacro:property name="hipW" value="0.045" />
+<xacro:property name="hipH" value="0.128" />
+<xacro:property name="hipSide" value="0.07" />
+<xacro:property name="hip_center_origin_L" value="0.028" />
+<!-- Knee -->
+<xacro:property name="knee_gearD" value="0.05" />
 <!-- leg -->
 <xacro:property name="legD" value="0.041" />
+<!-- Link3 -->
+<xacro:property name="link3_angle_limit" value="2.229" />
+<xacro:property name="footD" value="0.045" />
 <!-- Actuator -->
 <xacro:property name="actuator_nudge" value="0.00666" />
@@ -145,10 +153,10 @@
     <origin rpy="0 ${pi/2} 0" xyz="${L23/2} 0 0"/>
   </collision>
-  <!-- <collision name="link2_unit">
-    <geometry>
-      <cylinder radius="${actuator_diameter/2+connectorL_1}" length="${hipW+actuator3_wt_connectorL}"/>
-    </geometry>
-    <origin rpy="0 0 0" xyz="0 0 ${-(actuator3_wt_connectorL/2)}"/>
-  </collision> -->
+  <collision name="link2_hip">
+    <geometry>
+      <box size="${hipH} ${hipSide} ${hipW}" />
+    </geometry>
+    <origin rpy="0 0 0" xyz="${hip_center_origin_L} 0 0"/>
+  </collision>
   <inertial>
     <mass value="0.94987" />
@@ -169,4 +177,59 @@
   <origin rpy = "${pi/2} ${pi/2} 0" xyz="0 ${-L12}  0"/>
 </joint>
+  <!-- Link 3  -->
+<link name="link3">
+  <visual>
+    <geometry>
+        <mesh scale=".001 .001 .001" filename="package://leg_description/meshes/link3.STL" />
+    </geometry>
+    <origin rpy="0 0 0" xyz="0 0 0"/>
+    <material name="grey"/>
+  </visual>
+  <collision name="link3_leg">
+    <geometry>
+      <cylinder radius="${legD/2}" length="${L3E- (footD/2) }"/>
+    </geometry>
+    <origin rpy="0 ${pi/2} 0" xyz="${(L3E- (footD/2) )/2  } 0 0"/>
+  </collision>
+  <collision name="link3_knee">
+    <geometry>
+      <cylinder radius="${knee_gearD/2}" length="${legD }"/>
+    </geometry>
+    <origin rpy="0 0 0" xyz="0 0 0"/>
+  </collision>
+  <collision name="link3_foot">
+    <geometry>
+      <sphere radius="${footD/2}"/>
+    </geometry>
+    <origin rpy="0 0 0" xyz="${ L3E- footD/2  } 0 0"/>
+  </collision>
+  <inertial>
+    <mass value="0.36814" />
+    <inertia
+    ixx="8.8159e-05"
+    ixy="0"
+    ixz="0"
+    iyy="0.003793802"
+    iyz="0"
+    izz="0.003804351" />
+    <origin rpy="0 0 0" xyz="0.10653 0 0" />
+  </inertial>
+</link>
+<joint name="link2_to_link3" type="revolute">
+  <parent link="link2"/>
+  <child link="link3"/>
+  <axis rpy = "0 0 0" xyz="0 0 1"/>
+  <origin rpy = "0 0 0" xyz="${L23} 0  0"/>
+  <limit lower="${-link3_angle_limit}" upper="${link3_angle_limit}" effort="${effort_limit}" velocity="${velocity_limit}" />
+</joint>
+<transmission name="link2_link3_trans">
+    <type>transmission_interface/SimpleTransmission</type>
+    <actuator name="$motor3">
+      <mechanicalReduction>10</mechanicalReduction>
+    </actuator>
+    <joint name="link2_to_link3">
+      <hardwareInterface>hardware_interface/EffortJointInterface</hardwareInterface>
+    </joint>
+  </transmission>
 <transmission name="link1_link2_trans">
     <type>transmission_interface/SimpleTransmission</type>

Commit message: added positive products of  inertia

File: leg_description/urdf/my_leg.xacro (robot description, xacro)
@@ -47,18 +47,8 @@
 <xacro:property name="link1_total_mid_originL" value="${link1_total_length/2 - ( actuator_total_width - actuator_cylinder_width/2 - actuator_nudge) }" />
 <!-- Actuator Limits -->
-<xacro:property name="velocity_limit" value="398" />
+<xacro:property name="velocity_limit" value="388.4" />
 <xacro:property name="maxCurrent" value="13.36" />
-<xacro:property name="motorConstantKt" value="0.8" />
+<xacro:property name="motorConstantKt" value="0.0754" />
 <xacro:property name="effort_limit" value="${maxCurrent*motorConstantKt}" />
-<!-- Moment of inertia -->
-<xacro:macro name="default_inertial" params="mass xl yl zl *Dorigin">
-    <inertial>
-            <mass value="${mass}" />
-            <inertia ixx="${ mass * ( yl*yl + zl*zl ) / 12 }" ixy="0.0" ixz="0.0"
-                     iyy="${ mass * ( xl*xl + zl*zl ) / 12 }" iyz="0.0"
-                     izz="${ mass * ( yl*yl + xl*xl ) / 12 }" />
-            <xacro:insert_block name="Dorigin" />
-    </inertial>
-</xacro:macro>
 <!-- Addin objects: -->
 <link name="world"/>
@@ -111,11 +101,11 @@
   </collision>
   <inertial>
-    <mass value="1.14058" />
+    <mass value="0.4759" />
     <inertia
     ixx="0.000576572"
-    ixy="-1.091449e-05"
-    ixz="4.096e-06"
+    ixy="1.091449e-05"
+    ixz="-4.096e-06"
     iyy="0.000825053"
-    iyz="3.018e-06"
+    iyz="-3.018e-06"
     izz="0.000391889" />
     <origin rpy="0 0 0" xyz="-0.00083 -0.00061 0.01032" />
@@ -163,8 +153,8 @@
     <inertia
     ixx="0.001561735"
-    ixy="1.2537e-05"
-    ixz="0.000843757"
+    ixy="-1.2537e-05"
+    ixz="-0.000843757"
     iyy="0.005174717"
-    iyz="1.72e-05"
+    iyz="-1.72e-05"
     izz="0.004776989" />
     <origin rpy="0 0 0" xyz="0.03158 -0.00042 -0.02813" />
@@ -177,5 +167,14 @@
   <origin rpy = "${pi/2} ${pi/2} 0" xyz="0 ${-L12}  0"/>
 </joint>
-  <!-- Link 3  -->
+<transmission name="link1_link2_trans">
+    <type>transmission_interface/SimpleTransmission</type>
+    <actuator name="$motor2">
+      <mechanicalReduction>10</mechanicalReduction>
+    </actuator>
+    <joint name="link1_to_link2">
+      <hardwareInterface>hardware_interface/EffortJointInterface</hardwareInterface>
+    </joint>
+</transmission>
+<!-- Link 3  -->
 <link name="link3">
   <visual>
@@ -231,14 +230,5 @@
       <hardwareInterface>hardware_interface/EffortJointInterface</hardwareInterface>
     </joint>
-  </transmission>
-<transmission name="link1_link2_trans">
-    <type>transmission_interface/SimpleTransmission</type>
-    <actuator name="$motor2">
-      <mechanicalReduction>10</mechanicalReduction>
-    </actuator>
-    <joint name="link1_to_link2">
-      <hardwareInterface>hardware_interface/EffortJointInterface</hardwareInterface>
-    </joint>
-  </transmission>
+</transmission>
 <!-- Gazebo -->
 <gazebo>

Commit message: working effort position controllers for  full leg

File: leg_description/urdf/my_leg.xacro (robot description, xacro)
@@ -51,4 +51,8 @@
 <xacro:property name="motorConstantKt" value="0.0754" />
 <xacro:property name="effort_limit" value="${maxCurrent*motorConstantKt}" />
+<!-- Gear Reductions -->
+<xacro:property name="kr1" value="7" />
+<xacro:property name="kr2" value="10" />
+<xacro:property name="kr3" value="10" />
 <!-- Addin objects: -->
 <link name="world"/>
@@ -67,36 +71,4 @@
     </geometry>
     <origin rpy="0 0 0" xyz="0 0 ${AMOO/2}"/>
-  </collision>
-  <inertial>
-    <mass value="1.14058" />
-    <inertia
-    ixx="0.000576572"
-    ixy="-1.091449e-05"
-    ixz="4.096e-06"
-    iyy="0.000825053"
-    iyz="3.018e-06"
-    izz="0.000391889" />
-    <origin rpy="0 0 0" xyz="-0.00083 -0.00061 0.01032" />
-  </inertial>
-</link>
-<joint name="world_joint" type="fixed">
-  <parent link="world"/>
-  <child link="base_link"/>
-  <origin rpy="${pi/2} ${-pi/2} 0" xyz="${LB0} 0 ${BaseHeight}"/>
-</joint>
-<!-- Link 1  -->
-<link name="link1">
-  <visual>
-    <geometry>
-        <mesh scale=".001 .001 .001" filename="package://leg_description/meshes/link1.STL" />
-    </geometry>
-    <origin rpy="0 0 0" xyz="0 0 0"/>
-    <material name="grey"/>
-  </visual>
-  <collision>
-    <geometry>
-      <cylinder radius="${actuator_diameter/2+connectorL_1}" length="${link1_total_length}"/>
-    </geometry>
-    <origin rpy="${pi/2} 0 0" xyz="0  ${-link1_total_mid_originL} 0"/>
   </collision>
   <inertial>
@@ -112,9 +84,41 @@
   </inertial>
 </link>
+<joint name="world_joint" type="fixed">
+  <parent link="world"/>
+  <child link="base_link"/>
+  <origin rpy="${pi/2} ${-pi/2} 0" xyz="${LB0} 0 ${BaseHeight}"/>
+</joint>
+<!-- Link 1  -->
+<link name="link1">
+  <visual>
+    <geometry>
+        <mesh scale=".001 .001 .001" filename="package://leg_description/meshes/link1.STL" />
+    </geometry>
+    <origin rpy="0 0 0" xyz="0 0 0"/>
+    <material name="grey"/>
+  </visual>
+  <collision>
+    <geometry>
+      <cylinder radius="${actuator_diameter/2+connectorL_1}" length="${link1_total_length}"/>
+    </geometry>
+    <origin rpy="${pi/2} 0 0" xyz="0  ${-link1_total_mid_originL} 0"/>
+  </collision>
+  <inertial>
+    <mass value="0.4759" />
+    <inertia
+    ixx="0.000576572"
+    ixy="1.091449e-05"
+    ixz="-4.096e-06"
+    iyy="0.000825053"
+    iyz="-3.018e-06"
+    izz="0.000391889" />
+    <origin rpy="0 0 0" xyz="-0.00083 -0.00061 0.01032" />
+  </inertial>
+</link>
 <joint name="base_to_link1" type="revolute">
   <parent link="base_link"/>
   <child link="link1"/>
   <axis rpy = "0 0 0" xyz="0 0 1"/>
-  <limit lower="${-pi/2}" upper="${pi/2}" effort="${effort_limit}" velocity="${velocity_limit}" />
+  <limit lower="${-pi/2}" upper="${pi/2}" effort="${effort_limit*kr1}" velocity="${velocity_limit/kr1}" />
   <origin rpy = "0 0 0" xyz="0 0 ${-L01}"/>
 </joint>
@@ -122,5 +126,5 @@
     <type>transmission_interface/SimpleTransmission</type>
     <actuator name="motor1">
-      <mechanicalReduction>7</mechanicalReduction>
+      <mechanicalReduction>${kr1}</mechanicalReduction>
     </actuator>
     <joint name="base_to_link1">
@@ -166,9 +170,10 @@
   <axis rpy = "0 0 0" xyz="0 0 1"/>
   <origin rpy = "${pi/2} ${pi/2} 0" xyz="0 ${-L12}  0"/>
+  <limit effort="${effort_limit*kr2}" velocity="${velocity_limit/kr2}" />
 </joint>
 <transmission name="link1_link2_trans">
     <type>transmission_interface/SimpleTransmission</type>
     <actuator name="motor2">
-      <mechanicalReduction>10</mechanicalReduction>
+      <mechanicalReduction>${kr2}</mechanicalReduction>
     </actuator>
     <joint name="link1_to_link2">
@@ -220,10 +225,10 @@
   <axis rpy = "0 0 0" xyz="0 0 1"/>
   <origin rpy = "0 0 0" xyz="${L23} 0  0"/>
-  <limit lower="${-link3_angle_limit}" upper="${link3_angle_limit}" effort="${effort_limit}" velocity="${velocity_limit}" />
+  <limit lower="${-link3_angle_limit}" upper="${link3_angle_limit}" effort="${effort_limit*kr3}" velocity="${velocity_limit/kr3}" />
 </joint>
 <transmission name="link2_link3_trans">
     <type>transmission_interface/SimpleTransmission</type>
     <actuator name="motor3">
-      <mechanicalReduction>10</mechanicalReduction>
+      <mechanicalReduction>${kr3}</mechanicalReduction>
     </actuator>
     <joint name="link2_to_link3">
@@ -231,4 +236,9 @@
     </joint>
 </transmission>
+<!-- Gazebo references -->
+<gazebo reference="base_link" >
+  <material> Gazebo/Blue </material>
+  <kinematic> true </kinematic>
+</gazebo>
 <!-- Gazebo -->
 <gazebo>

Commit message: changed names on files

File: leg_description/urdf/my_leg.xacro (robot description, xacro)
@@ -241,4 +241,47 @@
   <kinematic> true </kinematic>
 </gazebo>
+<gazebo reference="link1" >
+  <material> Gazebo/Grey  </material>
+</gazebo>
+<gazebo reference="link2" >
+  <material> Gazebo/Grey  </material>
+</gazebo>
+<gazebo reference="link3" >
+  <material> Gazebo/Orange </material>
+  <!-- <collision>
+    <surface>
+      <friction>
+      <torsional>
+        <coefficient> 0 </coefficient>
+      </torsional>
+        <ode>
+          <mu>0.7</mu>
+          <mu2>1e-3</mu2>
+        </ode>
+      </friction>
+      <contact>
+        <ode>
+            <kp>1e4</kp>
+            <kd>1e2</kd>
+            <max_vel>100</max_vel>
+        </ode>
+      </contact>
+    </surface>
+  </collision> -->
+  <sensor type="contact" name="wall_contact_sensor">
+        <update_rate>1000.0</update_rate>
+        <always_on>1</always_on>
+        <contact>
+          <collision>link3_foot_collision_2</collision>
+          <topic>/link3_foot_collision</topic>
+        </contact>
+        <plugin name="gazebo_ros_bumper_controller" filename="libgazebo_ros_bumper.so">
+          <alwaysOn>true</alwaysOn>
+          <updateRate>1000.0</updateRate>
+          <bumperTopicName>/end_effector_collision</bumperTopicName>
+          <!-- <frameName></frameName> -->
+        </plugin>
+      </sensor>
+</gazebo>
 <!-- Gazebo -->
 <gazebo>

Commit message: expected forces, publishing transformed force

File: leg_description/urdf/my_leg.xacro (robot description, xacro)
@@ -249,5 +249,5 @@
 <gazebo reference="link3" >
   <material> Gazebo/Orange </material>
-  <!-- <collision>
+  <collision>
     <surface>
       <friction>
@@ -257,5 +257,5 @@
         <ode>
           <mu>0.7</mu>
-          <mu2>1e-3</mu2>
+          <!-- <mu2>1e-3</mu2> -->
         </ode>
       </friction>
@@ -268,5 +268,5 @@
       </contact>
     </surface>
-  </collision> -->
+  </collision>
   <sensor type="contact" name="wall_contact_sensor">
         <update_rate>1000.0</update_rate>
@@ -280,5 +280,5 @@
           <updateRate>1000.0</updateRate>
           <bumperTopicName>/end_effector_collision</bumperTopicName>
-          <!-- <frameName></frameName> -->
+          <frameName>world</frameName>
         </plugin>
       </sensor>

Commit message: changed L3E to 223 ( removed L3E-footD/2

File: leg_description/urdf/my_leg.xacro (robot description, xacro)
@@ -21,5 +21,5 @@
 <xacro:property name="L12" value="0.11208" />
 <xacro:property name="L23" value="0.2531" />
-<xacro:property name="L3E" value="0.2455" />
+<xacro:property name="L3E" value="0.223" />
 <!-- Connectors -->
 <xacro:property name="connectorL_1" value="0.004" />
@@ -194,5 +194,5 @@
       <cylinder radius="${legD/2}" length="${L3E- (footD/2) }"/>
     </geometry>
-    <origin rpy="0 ${pi/2} 0" xyz="${(L3E- (footD/2) )/2  } 0 0"/>
+    <origin rpy="0 ${pi/2} 0" xyz="${L3E/2  } 0 0"/>
   </collision>
   <collision name="link3_knee">
@@ -206,5 +206,5 @@
       <sphere radius="${footD/2}"/>
     </geometry>
-    <origin rpy="0 0 0" xyz="${ L3E- footD/2  } 0 0"/>
+    <origin rpy="0 0 0" xyz="${ L3E } 0 0"/>
   </collision>
   <inertial>
