Commit message: changed colors

File: leg_description/urdf/my_leg.xacro (robot description, xacro)
@@ -13,4 +13,7 @@
 <material name="DarkGrey">
   <color rgba="0.3 0.3 0.3 1"/>
+</material>
+<material name="orange">
+  <color rgba="1 0.5 0 1"/>
 </material>
 <!-- Defining macros -->
@@ -64,5 +67,5 @@
     </geometry>
     <origin rpy="0 0 0" xyz="0 0 0"/>
-    <material name="DarkGrey"/>
+    <material name="blue"/>
   </visual>
   <collision>
@@ -188,5 +191,5 @@
     </geometry>
     <origin rpy="0 0 0" xyz="0 0 0"/>
-    <material name="grey"/>
+    <material name="orange"/>
   </visual>
   <collision name="link3_leg">
@@ -245,5 +248,5 @@
 </gazebo>
 <gazebo reference="link2" >
-  <material> Gazebo/Grey  </material>
+  <material> Gazebo/DarkGrey  </material>
 </gazebo>
 <gazebo reference="link3" >
